File: hardware/PCB/Sensor_Plug_PCB.brd (EAGLE design)
At the start: 50 x 20 mm, 58 parts, among them IC1 MPRLS0025PA, IC2 EPS32-PICO-MINI-02, IC3 LIS3MDL, IC4 CP2102N-A02-GQFN24, IC5 TPS63031, IC6 MCP73831-DFN8, IC7 MAX17048, IC8 LSM6DSOX, J2 -, Q1 PMOS-SI2333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

Commit message: Change R5 to reduce charge current
Charge current was too ambitious leading to excessive heating during charging. This fixes the heat issue.
Parts:
- R4: value 2.0k -> 5.0k
Changed lines of the file:
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@@
 <attribute name="NAME" x="11.3" y="1.762" locked="yes" size="0.6096" layer="25" font="vector" ratio="20" align="bottom-center"/>
 </element>
-<element name="R4" library="Std Parts Library" library_urn="urn:adsk.wipprod:fs.file:vf.17mASCXCRkiwv_UU5McLmg" package="R0603" value="2.0k" x="2.413" y="14.859" smashed="yes">
+<element name="R4" library="Std Parts Library" library_urn="urn:adsk.wipprod:fs.file:vf.17mASCXCRkiwv_UU5McLmg" package="R0603" value="5.0k" x="2.413" y="14.859" smashed="yes">
 <attribute name="NAME" x="0.762" y="14.7101" size="0.6096" layer="25" font="vector" ratio="20" align="bottom-center"/>
 <attribute name="VALUE" x="4.064" y="16.3369" size="0.6096" layer="27" font="vector" ratio="20" align="top-center"/>

Commit message: new PCB revision
Parts:
- removed C14: 100nF, Std Parts Library:C0603
- removed I1: LPS3015-152 - 1.5µH, Std Parts Library:LPS3015
- removed IC7: MAX17048, Std Parts Library:DFN8_2X2
- added R13, R14: 200k, Std Parts Library:R0603
- added R17, R18: 100k, Std Parts Library:R0603
- C4: value 100nF -> 1uF
- IC5: value TPS63031 -> BU33SD5WG; device Std Parts Library:R-PWSON-N10 -> Std Parts Library:SOT23-5
- R3: value 1k -> 470
- moved M2 3.81 mm to (20.1, 17.5)
- moved D2 3.56 mm to (15.0, 17.7)
- moved C17 2.54 mm to (15.0, 13.3)
- moved C4 2.48 mm to (38.1, 7.24), turned to 90 degrees
- moved C7 1.05 mm to (25.0, 13.3)
- moved C13 1.05 mm to (19.1, 13.3)
- moved IC5 1.02 mm to (22.1, 13.2), turned to 0 degrees
- moved B1 0.25 mm to (46.7, 7.88)
Connections:
- removed net !BAT_ALRT: IC2.P$16, IC7.5
- removed net N$7: C14.2, IC5.6, IC5.8
- removed net N$8: I1.1, IC5.4
- removed net N$9: I1.2, IC5.2
- removed net VIN: C13.2, D4.C, IC5.5, Q1.2
- new net BAT_SENSE: C4.2, IC2.P$10, R13.1, R14.2
- new net N$2: C13.2, D4.C, IC5.1, IC5.3, Q1.2
- net +3V3: now also IC5.5; no longer IC5.1, IC5.10
- net GND: now also IC5.2, R14.1, R17.1, R18.1; no longer C14.1, IC5.11, IC5.3, IC5.7, IC5.9, IC7.1, IC7.4, IC7.6, IC7.9
- net MPR_EOC: now also IC2.P$9; no longer IC2.P$10
- net MPR_RST: now also IC2.P$20
- net SCL: no longer IC7.7
- net SDA: no longer IC7.8
- net VBAT: now also R13.2; no longer C4.2, IC7.2, IC7.3
- net VIBRATE0: now also R18.2
- net VIBRATE1: now also IC2.P$27, R17.2; no longer IC2.P$20
Routing:
- net MPR_RST: track 0.00 -> 29.4 mm, vias 0 -> 2
- net N$2: track 0.00 -> 23.9 mm
- net VIN: track 21.2 -> 0.00 mm
- net !BAT_ALRT: track 14.6 -> 0.00 mm, vias 2 -> 0
- net BAT_SENSE: track 0.00 -> 10.9 mm, vias 0 -> 2
- net N$7: track 3.55 -> 0.00 mm
- net VIBRATE1: track 20.1 -> 16.5 mm
- net +3V3: track 45.6 -> 42.7 mm, vias 4 -> 2
- net N$20: track 12.9 -> 15.6 mm
- net SCL: track 40.9 -> 38.4 mm
- net SDA: track 38.7 -> 36.9 mm, vias 4 -> 3
- net VIBRATE0: track 11.2 -> 12.6 mm
- net VBAT: track 123.9 -> 125.0 mm
- net MAG_RDY: track 13.7 -> 14.6 mm
- net MPR_EOC: track 24.0 -> 24.9 mm
- added copper zone on layer 1, net N$2
- removed copper zone on layer 1, net N$8
- removed copper zone on layer 1, net N$9
- removed copper zone on layer 1, net VIN
Other:
- board text added: "Charge Current 200 mA"
- board text added: "v0.3"
- board text removed: "Charge Current 500 mA"
- board text removed: "v0.2"
