File: hardware/PCB/Sensor_Plug_PCB.sch (EAGLE design)
At the start: 58 parts, among them IC1 MPRLS0025PA, IC2 EPS32-PICO-MINI-02, IC3 LIS3MDL, IC4 CP2102N-A02-GQFN24, IC5 TPS63031, IC6 MCP73831-DFN8, IC7 MAX17048, IC8 LSM6DSOX, J2 -, Q1 PMOS-SI2333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

Commit message: Change R5 to reduce charge current
Charge current was too ambitious leading to excessive heating during charging. This fixes the heat issue.
Parts:
- R4: value 2.0k -> 5.0k
Other:
- note added: "5.0K = 200mA"
- note removed: "1.0K = 1000mA"
- note removed: "1.3K = 750mA"
Changed lines of the file:
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@@
 <part name="R3" library="Std Parts Library" library_urn="urn:adsk.wipprod:fs.file:vf.17mASCXCRkiwv_UU5McLmg" deviceset="R" device="-0603" value="1k"/>
 <part name="LED1" library="Std Parts Library" library_urn="urn:adsk.wipprod:fs.file:vf.17mASCXCRkiwv_UU5McLmg" deviceset="LED" device="-0603-SIDEVIEW"/>
-<part name="R4" library="Std Parts Library" library_urn="urn:adsk.wipprod:fs.file:vf.17mASCXCRkiwv_UU5McLmg" deviceset="R" device="-0603" value="2.0k"/>
+<part name="R4" library="Std Parts Library" library_urn="urn:adsk.wipprod:fs.file:vf.17mASCXCRkiwv_UU5McLmg" deviceset="R" device="-0603" value="5.0k"/>
 <part name="GND21" library="Std Parts Library" library_urn="urn:adsk.wipprod:fs.file:vf.17mASCXCRkiwv_UU5McLmg" deviceset="GND" device="" value="GND"/>
 <part name="C15" library="Std Parts Library" library_urn="urn:adsk.wipprod:fs.file:vf.17mASCXCRkiwv_UU5McLmg" deviceset="C" device="-0805" value="10uF"/>
@@
 <wire x1="287.02" y1="109.22" x2="388.62" y2="109.22" width="0.8128" layer="97" style="longdash"/>
 <text x="139.7" y="195.58" size="5.08" layer="97" font="custom" fontFamily="Arial Rounded MT Bold">IMU</text>
-<text x="274.32" y="243.84" size="1.778" layer="97">3.3K  = 300mA</text>
-<text x="274.32" y="241.3" size="1.778" layer="97">2.0K  = 500mA</text>
-<text x="274.32" y="236.22" size="1.778" layer="97">1.0K  = 1000mA</text>
-<text x="274.32" y="238.76" size="1.778" layer="97">1.3K  = 750mA</text>
+<text x="274.32" y="238.76" size="1.778" layer="97">3.3K  = 300mA</text>
+<text x="274.32" y="236.22" size="1.778" layer="97">2.0K  = 500mA</text>
 <text x="325.12" y="218.44" size="1.27" layer="97">I2C Adress: 0x6C</text>
 <text x="332.74" y="137.16" size="1.27" layer="97">I2C Adress: 0x18</text>
@@
 <text x="217.678" y="114.554" size="1.27" layer="97">I2C Adress: 0x6A</text>
 <text x="217.17" y="157.988" size="1.27" layer="97">I2C Adress: 0x1C</text>
+<text x="274.32" y="241.3" size="1.778" layer="97">5.0K  = 200mA</text>
 </plain>
 <instances>

Commit message: new PCB revision
Parts:
- removed C14: 100nF, Std Parts Library:C-0603
- removed I1: LPS3015-152 - 1.5µH, Std Parts Library:I-LPS3015
- removed IC7: MAX17048, Std Parts Library:MAX17048/9
- added R13, R14: 200k, Std Parts Library:R-0603
- added R17, R18: 100k, Std Parts Library:R-0603
- C4: value 100nF -> 1uF
- IC5: value TPS63031 -> BU33SD5WG; device Std Parts Library:TPS63031 -> Std Parts Library:LDO-3.3V
- R3: value 1k -> 470
Connections:
- removed net !BAT_ALRT: IC2.IO26, IC7.!ALRT
- removed net N$7: C14.2, IC5.EN, IC5.VINA
- removed net N$8: I1.1, IC5.L1
- removed net N$9: I1.2, IC5.L2
- removed net VIN: C13.2, D4.C, IC5.VIN, Q1.S
- new net BAT_SENSE: C4.2, IC2.I35, R13.1, R14.2
- new net N$2: C13.2, D4.C, IC5.EN, IC5.IN, Q1.S
- net +3V3: now also IC5.OUT; no longer IC5.FB, IC5.VOUT
- net GND: now also R14.1, R17.1, R18.1; no longer C14.1, IC5.PGND, IC5.PS/SYNC, IC7.CTG, IC7.GND, IC7.QSTRT
- net MPR_EOC: now also IC2.I34; no longer IC2.I35
- net MPR_RST: now also IC2.IO13
- net SCL: no longer IC7.SCL
- net SDA: no longer IC7.SDA
- net VBAT: now also R13.2; no longer C4.2, IC7.CELL, IC7.VDD
- net VIBRATE0: now also R18.2
- net VIBRATE1: now also IC2.IO7, R17.2; no longer IC2.IO13
Other:
- note removed: "I2C Adress: 0x6C"
- moved on the sheet: C13, C16, C4, C7, D1, M1, Q4G$1
